File: template/PUT_Motorsport_4_Layer/template.kicad_pcb (KiCad board)
At the start: 2 copper layers, 60 x 40 mm, 4 parts

Commit message: Add 4 layer template
Other:
- copper layers 2 -> 4
Changed lines of the file:
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@@
 (kicad_pcb (version 20221018) (generator pcbnew)
   (general
-    (thickness 1.6)
+    (thickness 1.565)
   )
   (paper "A4")
@@
   (layers
     (0 "F.Cu" signal)
+    (1 "In1.Cu" signal)
+    (2 "In2.Cu" signal)
     (31 "B.Cu" signal)
     (34 "B.Paste" user)
@@
       (layer "F.Mask" (type "Top Solder Mask") (color "#073A61CC") (thickness 0.01) (material "Liquid Ink") (epsilon_r 3.3) (loss_tangent 0))
       (layer "F.Cu" (type "copper") (thickness 0.035))
-      (layer "dielectric 1" (type "prepreg") (color "#505543FF") (thickness 1.51) (material "FR4") (epsilon_r 4.5) (loss_tangent 0.02))
+      (layer "dielectric 1" (type "prepreg") (color "#505543FF") (thickness 0.1) (material "FR4") (epsilon_r 4.5) (loss_tangent 0.02))
+      (layer "In1.Cu" (type "copper") (thickness 0.0175))
+      (layer "dielectric 2" (type "prepreg") (color "#505543FF") (thickness 1.24) (material "FR4") (epsilon_r 4.5) (loss_tangent 0.02))
+      (layer "In2.Cu" (type "copper") (thickness 0.0175))
+      (layer "dielectric 3" (type "prepreg") (color "#505543FF") (thickness 0.1) (material "FR4") (epsilon_r 4.5) (loss_tangent 0.02))
       (layer "B.Cu" (type "copper") (thickness 0.035))
       (layer "B.Mask" (type "Bottom Solder Mask") (color "#073A61CC") (thickness 0.01) (material "Liquid Ink") (epsilon_r 3.3) (loss_tangent 0))
@@
   )
   (dimension (type aligned) (layer "Dwgs.User")
-    (pts (xy 121 81) (xy 171 81))
-    (height -10)
-    (gr_text "50 mm" (at 146 71) (layer "Dwgs.User")
+    (pts (xy 116 78) (xy 176 78))
+    (height -7)
+    (gr_text "60 mm" (at 146 71) (layer "Dwgs.User")
       (effects (font (size 1 1) (thickness 0.15)))
     )
@@
   )
   (dimension (type aligned) (layer "Dwgs.User")
-    (pts (xy 171 81) (xy 171 111))
-    (height -10)
-    (gr_text "30 mm" (at 181 96 90) (layer "Dwgs.User")
+    (pts (xy 174 76) (xy 174 116))
+    (height -7)
+    (gr_text "40 mm" (at 181 96 90) (layer "Dwgs.User")
       (effects (font (size 1 1) (thickness 0.15)))
     )
